Commit message: Enhance simulation configuration and introduce dashboard for teleoperation
- Updated the `.env` file to include a GUI option for the Gazebo simulation, defaulting to headless mode.
- Modified `docker-compose` files to support the new dashboard service on port 8090, allowing for a web-based control interface.
- Added a new `robomaster_dashboard` package, including a web UI for teleoperation and integration with the arm control.
- Updated launch files to incorporate the dashboard, ensuring it operates alongside existing simulation components.
- Enhanced the `Makefile` to reflect changes in bringup commands and clarify usage instructions for the new dashboard feature.

File: ros2_ws/src/robomaster_description/urdf/camera.urdf.xacro (robot description, xacro)
@@ -96,4 +96,45 @@
         </sensor>
       </gazebo>
+      <!-- Dashboard top-down: follows the chassis from above. Pixels only —
+           no optical TF / apriltag use. Gazebo looks along +X, so pitch -90
+           aims the sensor at the floor. -->
+      <link name="${tf_prefix}overview_camera_link">
+        <inertial>
+          <origin xyz="0 0 0" rpy="0 0 0" />
+          <mass value="0.001" />
+          <inertia ixx="0.001" ixy="0" ixz="0" iyy="0.001" iyz="0" izz="0.001" />
+        </inertial>
+      </link>
+      <joint name="${tf_prefix}overview_camera_joint" type="fixed">
+        <origin xyz="0 0 2.0" rpy="0 -1.5708 0" />
+        <parent link="${tf_prefix}base_link" />
+        <child link="${tf_prefix}overview_camera_link" />
+      </joint>
+      <gazebo reference="${tf_prefix}overview_camera_joint">
+        <preserveFixedJoint>true</preserveFixedJoint>
+        <disableFixedJointLumping>true</disableFixedJointLumping>
+      </gazebo>
+      <gazebo reference="${tf_prefix}overview_camera_link">
+        <sensor name="overview_camera" type="camera">
+          <pose>0 0 0 0 0 0</pose>
+          <camera>
+            <horizontal_fov>1.5708</horizontal_fov>
+            <image>
+              <width>640</width>
+              <height>480</height>
+              <format>R8G8B8</format>
+            </image>
+            <clip>
+              <near>0.1</near>
+              <far>40.0</far>
+            </clip>
+          </camera>
+          <always_on>1</always_on>
+          <update_rate>15</update_rate>
+          <visualize>false</visualize>
+          <topic>camera/overview</topic>
+          <gz_frame_id>${tf_prefix}overview_camera_link</gz_frame_id>
+        </sensor>
+      </gazebo>
     </xacro:if>
   </xacro:macro>
