Commit message: Add robomaster_arm package for Cartesian arm and gripper control
- Introduced the `robomaster_arm` package, including action definitions for moving the arm and setting the gripper.
- Implemented kinematics for the arm in `arm_kinematics.py` to handle inverse and forward kinematics.
- Created launch files to facilitate simulation and control of the arm and gripper.
- Updated the `CMakeLists.txt` and `package.xml` to include necessary dependencies and installation instructions.
- Enhanced the URDF configurations for the arm and gripper to ensure accurate simulation representation.

File: ros2_ws/src/robomaster_description/urdf/arm.urdf.xacro (robot description, xacro)
@@ -1,109 +1,14 @@
 <?xml version="1.0"?>
 <robot xmlns:xacro="http://playerstage.sourceforge.net/gazebo/xmlschema/#xacro">
-  <!-- The EP arm is two parallelogram linkages: three servo axes (arm_1_joint,
-       rod_joint, rod_3_joint) plus five bars whose angles are fixed by loop
-       closures. URDF is a kinematic tree and cannot express a closed loop, so
-       this description used to declare the bars as free joints tagged <mimic>.
-       <mimic> is not a constraint, only a hint that joint_state_publisher and
-       recent ros2_control read, and SDFormat 12 drops it outright: Gazebo
-       Fortress therefore saw eight unconstrained frictionless zero-effort
-       hinges, and gravity swung them indefinitely.
-       Fortress cannot express the constraint by any other route either, since
-       gz-physics' DART backend has no closed-chain support and mimic joints
-       only arrived in SDFormat 14 / Gazebo Harmonic. So every joint whose value
-       is determined by a loop closure is welded here instead. At zero the CAD
-       assembly pose is exactly consistent, so the welded result is the correct
-       assembled shape; it has no degrees of freedom left to drift, and it
-       behaves identically on every solver, physics engine and machine.
-       robot_state_publisher still publishes all of these frames.
-       Nothing in this stack actuates the arm anyway: ros2_control drives the
-       four wheels only. Articulating it needs a simulator that can close the
-       loops, or a description rebuilt around one serial chain per parallelogram.
-       Nominal servo ranges, kept for whoever does that: arm_1_joint
-       [-0.274, 1.384], rod_joint [-0.799, 1.731], rod_3_joint [-0.347, 1.215] rad.
-       Every inertia below is computed from the link's collision mesh by
-       scripts/mesh_inertia.py; edit scripts/inertia_manifest.txt and rerun it
-       rather than hand-editing these numbers. -->
+  <!-- Serial-equivalent EP arm for Fortress.
+       The real mechanism is closed parallelograms that SDFormat 12 / DART cannot
+       constrain. This tree keeps the CAD meshes that move with the two driven
+       links and places the endpoint with a planar 2R chain matching the EP
+       Cartesian workspace (SDK robotic_arm moveto x y, in cm). Decorative
+       linkage bars that only make sense as loop members are omitted so they
+       do not float or disconnect when the arm moves.
+       Joint limits approximate the old servo ranges projected onto this chain.
+       Inertias from scripts/mesh_inertia.py / inertia_manifest.txt. -->
   <xacro:macro name="arm" params="tf_prefix=''">
-    <link name="${tf_prefix}arm_1_link">
-      <inertial>
-        <origin xyz="0.01205666 0.02230166 0.05887051" rpy="0 0 0" />
-        <mass value="0.056" />
-        <inertia ixx="8.49512e-05" ixy="-3.95594e-07" ixz="-2.11241e-06" iyy="6.62308e-05"
-          iyz="-1.5812e-06" izz="2.53281e-05" />
-      </inertial>
-      <visual name="arm_1">
-        <origin xyz="0.0073108 0.0184816 0.0437162" rpy="0 0 0" />
-        <geometry>
-          <mesh filename="package://robomaster_description/meshes/arm_1.dae" scale="1.0 1.0 1.0" />
-        </geometry>
-        <material name="metal" />
-      </visual>
-      <visual name="arm_1_cylinder">
-        <origin xyz="-0.0239031 0.0255713 -0.0368083" rpy="0 0 0" />
-        <geometry>
-          <mesh filename="package://robomaster_description/meshes/arm_1_cylinder.dae"
-            scale="1.0 1.0 1.0" />
-        </geometry>
-        <material name="metal" />
-      </visual>
-      <collision name="arm_1_collision">
-        <origin xyz="0.0065116 0.0213649 0.0639448" rpy="0 0 0" />
-        <geometry>
-          <mesh filename="package://robomaster_description/meshes/arm_1_collision.dae"
-            scale="1.0 1.0 1.0" />
-        </geometry>
-      </collision>
-    </link>
-    <!-- <link name="arm_2_dummy">
-    </link> -->
-    <link name="${tf_prefix}arm_2_link">
-      <inertial>
-        <origin xyz="0.03671166 -0.02033782 0.00391168" rpy="0 0 0" />
-        <mass value="0.08" />
-        <inertia ixx="6.08608e-05" ixy="-6.10762e-08" ixz="6.09701e-05" iyy="0.000165693"
-          iyz="3.71217e-08" izz="0.000151413" />
-      </inertial>
-      <visual name="arm_2">
-        <origin xyz="0.0256122 -0.020134 -0.001308" rpy="0 0 0" />
-        <geometry>
-          <mesh filename="package://robomaster_description/meshes/arm_2.dae" scale="1.0 1.0 1.0" />
-        </geometry>
-        <!-- <material name="metal"/> -->
-        <material name="Test">
-          <color rgba="0.0 0.0 0.0 1.0" />
-        </material>
-      </visual>
-      <visual name="arm_2_bar_1">
-        <origin xyz="7.62e-05 0.0010863 -0.0002509" rpy="0 0 0" />
-        <geometry>
-          <mesh filename="package://robomaster_description/meshes/arm_2_bar_1.dae"
-            scale="1.0 1.0 1.0" />
-        </geometry>
-        <material name="metal" />
-      </visual>
-      <visual name="arm_2_bar_2">
-        <origin xyz="-0.0423232 -0.0099192 0.0221971" rpy="0 0 0" />
-        <geometry>
-          <mesh filename="package://robomaster_description/meshes/arm_2_bar_2.dae"
-            scale="1.0 1.0 1.0" />
-        </geometry>
-        <material name="metal" />
-      </visual>
-      <collision name="arm_2_collision">
-        <origin xyz="0.0222614 -0.0202749 -0.008504" rpy="0 0 0" />
-        <geometry>
-          <mesh filename="package://robomaster_description/meshes/arm_2_collision.dae"
-            scale="1.0 1.0 1.0" />
-        </geometry>
-      </collision>
-    </link>
-    <!-- <link name="arm_base_attachment_link">
-      <inertial>
-        <origin xyz="0 0 0" rpy="0 0 0"/>
-        <mass value="0.001"/>
-        <inertia ixx="0.001" ixy="0" ixz="0" iyy="0.001" iyz="0" izz="0.001"/>
-      </inertial>
-    </link> -->
     <link name="${tf_prefix}arm_base_link">
       <inertial>
@@ -144,13 +49,73 @@
       </collision>
     </link>
-    <!-- Geometryless frames get a nominal point-mass inertia: small enough not
-         to perturb the body they weld into, large enough to stay positive
-         definite. -->
-    <link name="${tf_prefix}end_point_link">
+    <link name="${tf_prefix}arm_1_link">
       <inertial>
-        <origin xyz="0 0 0" rpy="0 0 0" />
-        <mass value="0.001" />
-        <inertia ixx="1e-09" ixy="0" ixz="0" iyy="1e-09" iyz="0" izz="1e-09" />
+        <origin xyz="0.01205666 0.02230166 0.05887051" rpy="0 0 0" />
+        <mass value="0.056" />
+        <inertia ixx="8.49512e-05" ixy="-3.95594e-07" ixz="-2.11241e-06" iyy="6.62308e-05"
+          iyz="-1.5812e-06" izz="2.53281e-05" />
       </inertial>
+      <visual name="arm_1">
+        <origin xyz="0.0073108 0.0184816 0.0437162" rpy="0 0 0" />
+        <geometry>
+          <mesh filename="package://robomaster_description/meshes/arm_1.dae" scale="1.0 1.0 1.0" />
+        </geometry>
+        <material name="metal" />
+      </visual>
+      <visual name="arm_1_cylinder">
+        <origin xyz="-0.0239031 0.0255713 -0.0368083" rpy="0 0 0" />
+        <geometry>
+          <mesh filename="package://robomaster_description/meshes/arm_1_cylinder.dae"
+            scale="1.0 1.0 1.0" />
+        </geometry>
+        <material name="metal" />
+      </visual>
+      <collision name="arm_1_collision">
+        <origin xyz="0.0065116 0.0213649 0.0639448" rpy="0 0 0" />
+        <geometry>
+          <mesh filename="package://robomaster_description/meshes/arm_1_collision.dae"
+            scale="1.0 1.0 1.0" />
+        </geometry>
+      </collision>
+    </link>
+    <link name="${tf_prefix}arm_2_link">
+      <inertial>
+        <origin xyz="0.03671166 -0.02033782 0.00391168" rpy="0 0 0" />
+        <mass value="0.08" />
+        <inertia ixx="6.08608e-05" ixy="-6.10762e-08" ixz="6.09701e-05" iyy="0.000165693"
+          iyz="3.71217e-08" izz="0.000151413" />
+      </inertial>
+      <visual name="arm_2">
+        <origin xyz="0.0256122 -0.020134 -0.001308" rpy="0 0 0" />
+        <geometry>
+          <mesh filename="package://robomaster_description/meshes/arm_2.dae" scale="1.0 1.0 1.0" />
+        </geometry>
+        <material name="Test">
+          <color rgba="0.0 0.0 0.0 1.0" />
+        </material>
+      </visual>
+      <visual name="arm_2_bar_1">
+        <origin xyz="7.62e-05 0.0010863 -0.0002509" rpy="0 0 0" />
+        <geometry>
+          <mesh filename="package://robomaster_description/meshes/arm_2_bar_1.dae"
+            scale="1.0 1.0 1.0" />
+        </geometry>
+        <material name="metal" />
+      </visual>
+      <visual name="arm_2_bar_2">
+        <origin xyz="-0.0423232 -0.0099192 0.0221971" rpy="0 0 0" />
+        <geometry>
+          <mesh filename="package://robomaster_description/meshes/arm_2_bar_2.dae"
+            scale="1.0 1.0 1.0" />
+        </geometry>
+        <material name="metal" />
+      </visual>
+      <collision name="arm_2_collision">
+        <origin xyz="0.0222614 -0.0202749 -0.008504" rpy="0 0 0" />
+        <geometry>
+          <mesh filename="package://robomaster_description/meshes/arm_2_collision.dae"
+            scale="1.0 1.0 1.0" />
+        </geometry>
+      </collision>
     </link>
     <link name="${tf_prefix}endpoint_bracket_link">
@@ -177,162 +142,11 @@
       </collision>
     </link>
-    <!-- <link name="rod_1_dummy">
-    </link> -->
-    <link name="${tf_prefix}rod_1_link">
+    <link name="${tf_prefix}end_point_link">
       <inertial>
-        <origin xyz="-0.04802565 0 0.03246364" rpy="0 0 0" />
-        <mass value="0.012" />
-        <inertia ixx="4.97769e-06" ixy="0" ixz="8.37868e-06" iyy="2.02607e-05" iyz="0"
-          izz="1.53005e-05" />
+        <origin xyz="0 0 0" rpy="0 0 0" />
+        <mass value="0.001" />
+        <inertia ixx="1e-09" ixy="0" ixz="0" iyy="1e-09" iyz="0" izz="1e-09" />
       </inertial>
-      <visual name="rod_1">
-        <origin xyz="-0.0479737 0 0.0301898" rpy="0 0 0" />
-        <geometry>
-          <mesh filename="package://robomaster_description/meshes/rod_1.dae" scale="1.0 1.0 1.0" />
-        </geometry>
-        <material name="metal" />
-      </visual>
-      <collision name="rod_1_collision">
-        <origin xyz="-0.0477809 0 0.0272644" rpy="0 0 0" />
-        <geometry>
-          <mesh filename="package://robomaster_description/meshes/rod_1_collision.dae"
-            scale="1.0 1.0 1.0" />
-        </geometry>
-      </collision>
     </link>
-    <!-- <link name="rod_2_dummy">
-      <inertial>
-        <origin xyz="0 0 0" rpy="0 0 0"/>
-        <mass value="0.001"/>
-        <inertia ixx="0.001" ixy="0" ixz="0" iyy="0.001" iyz="0" izz="0.001"/>
-      </inertial>
-    </link> -->
-    <link name="${tf_prefix}rod_2_link">
-      <inertial>
-        <origin xyz="-0.003175907 0 0.05794559" rpy="0 0 0" />
-        <mass value="0.012" />
-        <inertia ixx="2.00286e-05" ixy="0" ixz="-5.50685e-07" iyy="2.03218e-05" iyz="0"
-          izz="3.10675e-07" />
-      </inertial>
-      <visual name="rod_2">
-        <origin xyz="-0.0012722 0 0.0561361" rpy="0 0 0" />
-        <geometry>
-          <mesh filename="package://robomaster_description/meshes/rod_2.dae"
-            scale="1.0000004 1.0 0.9999998" />
-        </geometry>
-        <material name="metal" />
-      </visual>
-      <collision name="rod_2_collision">
-        <origin xyz="0.0011528 0 0.0549123" rpy="0 0 0" />
-        <geometry>
-          <mesh filename="package://robomaster_description/meshes/rod_2_collision.dae"
-            scale="1.0000004 1.0 0.9999998" />
-        </geometry>
-      </collision>
-    </link>
-    <!-- <link name="rod_3_dummy">
-      <inertial>
-        <origin xyz="0 0 0" rpy="0 0 0"/>
-        <mass value="0.001"/>
-        <inertia ixx="0.001" ixy="0" ixz="0" iyy="0.001" iyz="0" izz="0.001"/>
-      </inertial>
-    </link> -->
-    <link name="${tf_prefix}rod_3_link">
-      <inertial>
-        <origin xyz="-0.003713694 9.504091e-06 0.06138324" rpy="0 0 0" />
-        <mass value="0.012" />
-        <inertia ixx="2.01022e-05" ixy="0" ixz="-4.94278e-07" iyy="2.0411e-05" iyz="0"
-          izz="3.26386e-07" />
-      </inertial>
-      <visual name="rod_3">
-        <origin xyz="-0.0017304 0 0.0633558" rpy="0 0 0" />
-        <geometry>
-          <mesh filename="package://robomaster_description/meshes/rod_3.dae" scale="1.0 1.0 1.0" />
-        </geometry>
-        <material name="metal" />
-      </visual>
-      <collision name="rod_3_collision">
-        <origin xyz="0.0004696 9.5e-06 0.0561803" rpy="0 0 0" />
-        <geometry>
-          <mesh filename="package://robomaster_description/meshes/rod_3_collision.dae"
-            scale="1.0 1.0 1.0" />
-        </geometry>
-      </collision>
-    </link>
-    <link name="${tf_prefix}rod_link">
-      <inertial>
-        <origin xyz="-0.02068464 0.002379249 0.008827015" rpy="0 0 0" />
-        <mass value="0.011" />
-        <inertia ixx="1.3148e-06" ixy="0" ixz="1.84731e-06" iyy="5.21407e-06" iyz="0"
-          izz="3.97845e-06" />
-      </inertial>
-      <visual name="rod">
-        <origin xyz="-0.0261857 0.0022566 0.0121229" rpy="0 0 0" />
-        <geometry>
-          <mesh filename="package://robomaster_description/meshes/rod.dae" scale="1.0 1.0 1.0" />
-        </geometry>
-        <material name="metal" />
-      </visual>
-      <collision name="rod_collision">
-        <origin xyz="-0.02432 0.0022871 0.0136485" rpy="0 0 0" />
-        <geometry>
-          <mesh filename="package://robomaster_description/meshes/rod_collision.dae"
-            scale="1.0 1.0 1.0" />
-        </geometry>
-      </collision>
-    </link>
-    <!-- <link name="triangle_1_dummy">
-      <inertial>
-        <origin xyz="0 0 0" rpy="0 0 0"/>
-        <mass value="0.001"/>
-        <inertia ixx="0.001" ixy="0" ixz="0" iyy="0.001" iyz="0" izz="0.001"/>
-      </inertial>
-    </link> -->
-    <!-- <link name="triangle_2_dummy">
-    </link> -->
-    <link name="${tf_prefix}triangle_link">
-      <inertial>
-        <origin xyz="-0.01120213 0 0.0129844" rpy="0 0 0" />
-        <mass value="0.009" />
-        <inertia ixx="6.19224e-07" ixy="0" ixz="-1.62891e-08" iyy="2.7415e-06" iyz="0"
-          izz="2.13638e-06" />
-      </inertial>
-      <visual name="triangle">
-        <origin xyz="-0.0095953 0 0.0131247" rpy="0 0 0" />
-        <geometry>
-          <mesh filename="package://robomaster_description/meshes/triangle.dae" scale="1.0 1.0 1.0" />
-        </geometry>
-        <material name="metal" />
-      </visual>
-      <collision name="triangle_collision">
-        <origin xyz="-0.0091994 0 0.012377" rpy="0 0 0" />
-        <geometry>
-          <mesh filename="package://robomaster_description/meshes/triangle_collision.dae"
-            scale="1.0 1.0 1.0" />
-        </geometry>
-      </collision>
-    </link>
-    <!-- Servo axis. Welded: rod_2_link and triangle_link close loops around it. -->
-    <joint name="${tf_prefix}arm_1_joint" type="fixed">
-      <origin xyz="0.0103961 -0.0255713 0.030741" rpy="0 0 0" />
-      <parent link="${tf_prefix}arm_base_link" />
-      <child link="${tf_prefix}arm_1_link" />
-    </joint>
-    <!-- <joint name="arm_2_dummy" type="floating">
-      <origin xyz="-0.0419304 0.0028425 0.0218356" rpy="0 0 0"/>
-      <parent link="arm_2_link"/>
-      <child link="arm_2_dummy"/>
-    </joint> -->
-    <!-- Was: mimic of rod_3_joint, multiplier -1. -->
-    <joint name="${tf_prefix}arm_2_joint" type="fixed">
-      <origin xyz="0.0018704 0.0438659 0.1210238" rpy="0 0 0" />
-      <parent link="${tf_prefix}arm_1_link" />
-      <child link="${tf_prefix}arm_2_link" />
-    </joint>
-    <!-- <joint name="arm_base_attachment_joint" type="fixed">
-      <origin xyz="0 0.0010384 0.0906477" rpy="0 0 0"/>
-      <parent link="base_link"/>
-      <child link="arm_base_attachment_link"/>
-    </joint> -->
     <joint name="${tf_prefix}arm_base_joint" type="fixed">
       <origin xyz="0 0.0010384 0.0906477" rpy="0 0 0" />
@@ -340,9 +154,27 @@
       <child link="${tf_prefix}arm_base_link" />
     </joint>
-    <!-- <joint name="attachement_link" type="floating">
-      <origin xyz="0 0 0" rpy="0 0 0"/>
-      <parent link="arm_base_link"/>
-      <child link="attachement_link"/>
-    </joint> -->
+    <!-- Shoulder: rotates about +Y in the robot's sagittal plane. -->
+    <joint name="${tf_prefix}arm_1_joint" type="revolute">
+      <origin xyz="0.0103961 -0.0255713 0.030741" rpy="0 0 0" />
+      <parent link="${tf_prefix}arm_base_link" />
+      <child link="${tf_prefix}arm_1_link" />
+      <axis xyz="0 1 0" />
+      <limit lower="-0.274" upper="1.384" effort="5.0" velocity="2.0" />
+      <dynamics damping="0.1" friction="0.05" />
+    </joint>
+    <!-- Elbow. Length along this link to the EE is ~L2 for IK. -->
+    <joint name="${tf_prefix}arm_2_joint" type="revolute">
+      <origin xyz="0.0018704 0.0438659 0.1210238" rpy="0 0 0" />
+      <parent link="${tf_prefix}arm_1_link" />
+      <child link="${tf_prefix}arm_2_link" />
+      <axis xyz="0 1 0" />
+      <limit lower="-1.8" upper="0.35" effort="5.0" velocity="2.0" />
+      <dynamics damping="0.1" friction="0.05" />
+    </joint>
+    <joint name="${tf_prefix}endpoint_bracket_joint" type="fixed">
+      <origin xyz="0.1058557 0.006752 -0.0561093" rpy="0 0 0" />
+      <parent link="${tf_prefix}arm_2_link" />
+      <child link="${tf_prefix}endpoint_bracket_link" />
+    </joint>
     <joint name="${tf_prefix}end_point_joint" type="fixed">
       <origin xyz="0.0110125 -0.0270264 -0.0103816" rpy="0 0 0" />
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