Commit message: Add script for gripper diagnostics and update arm presets
- Introduced a new script `_tmp_grip2.sh` for listing ROS2 nodes, controllers, and hardware interfaces related to the gripper.
- Updated the "tuck" preset in `arm_kinematics.py` and `teleop_node.py` to adjust arm positioning for improved control.
- Modified the `arm_node.py` to ensure both gripper fingers receive the same command for consistent operation.
- Enhanced dashboard functionality to improve user interaction with the gripper controls.

File: ros2_ws/src/robomaster_description/urdf/gripper.urdf.xacro (robot description, xacro)
@@ -1,10 +1,8 @@
 <?xml version="1.0"?>
 <robot xmlns:xacro="http://playerstage.sourceforge.net/gazebo/xmlschema/#xacro">
-  <!-- Parallel-jaw approximation of the EP gripper. The real fingers are a
-       five-bar loop Fortress cannot close; instead each finger rides a
-       prismatic joint along ±Y. Mesh origins are the CAD assembly poses
-       (absolute in gripper_link) from the old welded chain. Command interface
-       stays gripper_m_joint in [-0.023, 0.001]; the right finger is driven as
-       the negation so open/close pinches instead of sliding in X. -->
+  <!-- Parallel-jaw approximation of the EP gripper. Proximal finger meshes stay
+       welded at the CAD pose on gripper_link; only the tips (link 7) ride
+       opposing prismatic joints along ±Y. Both joints take the same command
+       value (axes are opposite). Limits stay [-0.023, 0.001]. -->
   <xacro:macro name="gripper" params="tf_prefix=''">
     <link name="${tf_prefix}gripper_link">
@@ -30,12 +28,5 @@
         </geometry>
       </collision>
-    </link>
-    <!-- Left finger (+Y). Origins are CAD poses relative to gripper_link. -->
-    <link name="${tf_prefix}gripper_m_link">
-      <inertial>
-        <origin xyz="0.056 0.0174 -0.04" rpy="0 0 0" />
-        <mass value="0.01" />
-        <inertia ixx="1e-06" ixy="0" ixz="0" iyy="1e-06" iyz="0" izz="1e-06" />
-      </inertial>
+      <!-- Proximal left finger (fixed CAD pose). -->
       <visual name="left_gripper_1">
         <origin xyz="0.016288 0.0212844 -0.0399426" rpy="0 0 0" />
@@ -78,27 +69,5 @@
         <material name="EP_up.001" />
       </visual>
-      <visual name="left_gripper_7">
-        <origin xyz="0.056 0.0174005 -0.0399426" rpy="0 0 0" />
-        <geometry>
-          <mesh filename="package://robomaster_description/meshes/gripper_left_7.dae"
-            scale="1.0 1.0 1.0" />
-        </geometry>
-        <material name="EP_up.001" />
-      </visual>
-      <collision name="left_gripper_collision">
-        <origin xyz="0.0564138 0.0172595 -0.0695631" rpy="0 0 0" />
-        <geometry>
-          <mesh filename="package://robomaster_description/meshes/gripper_left_collision.dae"
-            scale="1.0 1.0 1.0" />
-        </geometry>
-      </collision>
-    </link>
-    <!-- Right finger (−Y via commanded negation of gripper_m_joint). -->
-    <link name="${tf_prefix}gripper_r_link">
-      <inertial>
-        <origin xyz="0.056 -0.0174 -0.04" rpy="0 0 0" />
-        <mass value="0.01" />
-        <inertia ixx="1e-06" ixy="0" ixz="0" iyy="1e-06" iyz="0" izz="1e-06" />
-      </inertial>
+      <!-- Proximal right finger (fixed CAD pose). -->
       <visual name="right_gripper_1">
         <origin xyz="0.0162882 -0.0210593 -0.0399426" rpy="0 0 0" />
@@ -141,4 +110,35 @@
         <material name="EP_up.001" />
       </visual>
+    </link>
+    <!-- Left tip (+Y). -->
+    <link name="${tf_prefix}gripper_m_link">
+      <inertial>
+        <origin xyz="0.056 0.0174 -0.04" rpy="0 0 0" />
+        <mass value="0.01" />
+        <inertia ixx="1e-06" ixy="0" ixz="0" iyy="1e-06" iyz="0" izz="1e-06" />
+      </inertial>
+      <visual name="left_gripper_7">
+        <origin xyz="0.056 0.0174005 -0.0399426" rpy="0 0 0" />
+        <geometry>
+          <mesh filename="package://robomaster_description/meshes/gripper_left_7.dae"
+            scale="1.0 1.0 1.0" />
+        </geometry>
+        <material name="EP_up.001" />
+      </visual>
+      <collision name="left_gripper_collision">
+        <origin xyz="0.0564138 0.0172595 -0.0695631" rpy="0 0 0" />
+        <geometry>
+          <mesh filename="package://robomaster_description/meshes/gripper_left_collision.dae"
+            scale="1.0 1.0 1.0" />
+        </geometry>
+      </collision>
+    </link>
+    <!-- Right tip (−Y via opposite joint axis). -->
+    <link name="${tf_prefix}gripper_r_link">
+      <inertial>
+        <origin xyz="0.056 -0.0174 -0.04" rpy="0 0 0" />
+        <mass value="0.01" />
+        <inertia ixx="1e-06" ixy="0" ixz="0" iyy="1e-06" iyz="0" izz="1e-06" />
+      </inertial>
       <visual name="right_gripper_7">
         <origin xyz="0.0711547 -0.0342395 -0.0399426" rpy="0 0 0" />
@@ -169,5 +169,4 @@
       <child link="${tf_prefix}gripper_link" />
     </joint>
-    <!-- 0.001 = open (wider), -0.023 = closed (pinch). Axis +Y. -->
     <joint name="${tf_prefix}gripper_m_joint" type="prismatic">
       <origin xyz="0 0 0" rpy="0 0 0" />
@@ -175,15 +174,14 @@
       <child link="${tf_prefix}gripper_m_link" />
       <axis xyz="0 1 0" />
-      <limit lower="-0.023" upper="0.001" effort="20.0" velocity="0.05" />
-      <dynamics damping="1.0" friction="0.5" />
+      <limit lower="-0.023" upper="0.001" effort="40.0" velocity="0.08" />
+      <dynamics damping="0.05" friction="0.0" />
     </joint>
-    <!-- Commanded as -gripper_m_joint so fingers move toward each other. -->
     <joint name="${tf_prefix}gripper_r_joint" type="prismatic">
       <origin xyz="0 0 0" rpy="0 0 0" />
       <parent link="${tf_prefix}gripper_link" />
       <child link="${tf_prefix}gripper_r_link" />
-      <axis xyz="0 1 0" />
-      <limit lower="-0.001" upper="0.023" effort="20.0" velocity="0.05" />
-      <dynamics damping="1.0" friction="0.5" />
+      <axis xyz="0 -1 0" />
+      <limit lower="-0.023" upper="0.001" effort="40.0" velocity="0.08" />
+      <dynamics damping="0.05" friction="0.0" />
     </joint>
     <joint name="${tf_prefix}gripper_joint_t" type="fixed">

Commit message: Remove temporary gripper diagnostics script and update arm control logic
- Deleted the `_tmp_grip2.sh` script used for gripper diagnostics.
- Enhanced the `MoveArm.action` file to include joint control options for the arm.
- Updated `arm_kinematics.py` to improve preset definitions for arm positioning.
- Modified `arm_node.py` to hold gripper commands more reliably during operation.
- Adjusted dashboard and teleop scripts to reflect new arm control capabilities and preset structures.
- Improved camera feed handling in the dashboard for a more stable user experience.

File: ros2_ws/src/robomaster_description/urdf/gripper.urdf.xacro (robot description, xacro)
@@ -126,9 +126,9 @@
         <material name="EP_up.001" />
       </visual>
+      <!-- Box pads: mesh collisions were jamming the prismatic tips in Gazebo. -->
       <collision name="left_gripper_collision">
-        <origin xyz="0.0564138 0.0172595 -0.0695631" rpy="0 0 0" />
+        <origin xyz="0.062 0.017 -0.045" rpy="0 0 0" />
         <geometry>
-          <mesh filename="package://robomaster_description/meshes/gripper_left_collision.dae"
-            scale="1.0 1.0 1.0" />
+          <box size="0.025 0.012 0.02" />
         </geometry>
       </collision>
@@ -150,8 +150,7 @@
       </visual>
       <collision name="right_gripper_7_collision">
-        <origin xyz="0.0561863 -0.0173908 -0.0695631" rpy="0 0 0" />
+        <origin xyz="0.062 -0.017 -0.045" rpy="0 0 0" />
         <geometry>
-          <mesh filename="package://robomaster_description/meshes/right_gripper_7_collision.dae"
-            scale="1.0 1.0 1.0" />
+          <box size="0.025 0.012 0.02" />
         </geometry>
       </collision>
